Commit message: Fixed URDF gofa + Single arm Yumi. Merged in ine pkg. Removed Yumi URDF

File: robots_description/Grippers/YumiServoGripper/yumi_servo_gripper.transmission.xacro (robot description, xacro)
@@ -2,12 +2,12 @@
 <robot name="yumi_servo_gripper" xmlns:xacro="http://www.ros.org/wiki/xacro">
   <xacro:macro name="yumi_servo_gripper_transmission" params="name hardware_interface">
-   <transmission name="${name}_tran">
+    <transmission name="${name}_tran">
       <type>transmission_interface/SimpleTransmission</type>
       <joint name="${name}_joint">
-	<hardwareInterface>${hardware_interface}</hardwareInterface>
+        <hardwareInterface>${hardware_interface}</hardwareInterface>
       </joint>
       <actuator name="${name}_motor">
-	<hardwareInterface>${hardware_interface}</hardwareInterface>
-	<mechanicalReduction>1</mechanicalReduction>
+        <hardwareInterface>${hardware_interface}</hardwareInterface>
+        <mechanicalReduction>1</mechanicalReduction>
       </actuator>
     </transmission>

File: robots_description/Util/utilities.xacro (robot description, xacro)
@@ -6,14 +6,14 @@
   <!--Cuboid-->
   <xacro:macro name="cuboid_inertia" params="width height length mass">
-    <inertia ixx="${mass * (height * height + length * length) / 12)}"
-             iyy="${mass * (width * width + length * length) / 12)}"
-             izz="${mass * (width * width + height * height) / 12)}"
+    <inertia ixx="${mass * (height * height + length * length) / 12}"
+             iyy="${mass * (width * width + length * length) / 12}"
+             izz="${mass * (width * width + height * height) / 12}"
              ixy="0" iyz="0" ixz="0"/>
   </xacro:macro>
   <!--Cylinder: length is along the y-axis! -->
   <xacro:macro name="cylinder_inertia" params="radius length mass">
-    <inertia ixx="${mass * (3 * radius * radius + length * length) / 12)}"
-             iyy="${mass * radius* radius / 2)}"
-             izz="${mass * (3 * radius * radius + length * length) / 12)}"
+    <inertia ixx="${mass * (3 * radius * radius + length * length) / 12}"
+             iyy="${mass * radius* radius / 2}"
+             izz="${mass * (3 * radius * radius + length * length) / 12}"
              ixy="0" iyz="0" ixz="0"/>
   </xacro:macro>

File: robots_description/xacro/robot.urdf.xacro (robot description, xacro)
@@ -1,24 +1,43 @@
 <?xml version="1.0"?>
-<robot xmlns:xacro="http://www.ros.org/wiki/xacro" name="robot" >
-    <xacro:arg name="robot"   default="gofa"/>
-    <xacro:property name="robot" value="$(arg robot)"/>
+<robot xmlns:xacro="http://www.ros.org/wiki/xacro" name="robot">
+    <!-- Parameters -->
+    <arg name="name"                    default="gofa" />
+    <xacro:arg name="robot"              default="$(arg name)" />
+    <xacro:arg name="hardware_interface" default="PositionJointInterface" />
+    <xacro:arg name="gripper_interface"  default="EffortJointInterface" />
+    <xacro:arg name="yumi_setup"         default="default" />
+    <xacro:property name="robot"              value="$(arg robot)" />
+    <xacro:property name="hardware_interface" value="$(arg hardware_interface)" />
+    <xacro:property name="gripper_interface"  value="$(arg gripper_interface)" />
+    <!-- World fixed joint -->
+    <link name="world" />
     <!-- Robot -->
+    <!-- Gofa -->
     <xacro:if value="${robot == 'gofa'}">
-        <xacro:include filename="$(find robots_description)/xacro/gofa.urdf.xacro" />
+        <xacro:include filename="$(find robots_description)/xacro/Gofa/gofa.urdf.xacro" />
         <xacro:gofa parent="world" child="flange">
-            <origin xyz="0 0 0" rpy="0 0 0"/>
+            <origin xyz="0 0 0" rpy="0 0 0" />
         </xacro:gofa>
+        <!-- Gripper -->
     </xacro:if>
-    <!--xacro:if value="${robot == 'yumi'}">
-        <xacro:include filename="$(find robots_description)/xacro/yumi.urdf.xacro" />
-    </xacro:if-->
-    <!-- Grippers
-    <xacro:if value="${gr == 'robotiq_2f'}">
-        <xacro:include filename="$(find dsr_description)/xacro/robotiq_2f.urdf.xacro" />
+    <!-- Single Yumi -->
+    <xacro:if value="${robot == 'yumi_single_arm'}">
+        <!-- Import Rviz colors -->
+        <xacro:include filename="$(find robots_description)/Util/materials.xacro" />
+        <!-- Import utilities -->
+        <xacro:include filename="$(find robots_description)/Util/utilities.xacro" />
+        <!--Import
+        the single yumi macro -->
+        <xacro:include filename="$(find robots_description)/xacro/YumiSingleArm/single_yumi.xacro" />
+        <!--Import
+        the yumi servo gripper macro -->
+        <xacro:include filename="$(find robots_description)/Grippers/YumiServoGripper/yumi_servo_gripper.xacro" />
+        <xacro:single_yumi parent="world" hardware_interface="${hardware_interface}">
+            <origin xyz="0 0 0" rpy="0 0 0" />
+        </xacro:single_yumi>
+        <!-- Gripper -->
+        <xacro:yumi_servo_gripper name="gripper" parent="link_7" hardware_interface="${gripper_interface}">
+            <origin xyz="0 0 0.007" rpy="0 0 ${PI}" />
+        </xacro:yumi_servo_gripper>
     </xacro:if>
-    <xacro:if value="${gr == 'GripperCamozzi'}">
-        <xacro:include filename="$(find dsr_description)/xacro/GripperCamozzi/GripperCamozzi.urdf.xacro" />
-    </xacro:if> -->
-    <!-- World fixed joint-->
-    <link name="world" />
 </robot>
