Commit message: Fixed Flange Orientation

File: robots_description/xacro/Gofa/gofa.urdf.xacro (robot description, xacro)
@@ -145,5 +145,5 @@
 		</link>
 		<joint name="$(arg 6th_link_name)_to_${child}" type="fixed">
-			<origin xyz="0.033599981 0 0" rpy="0 0 0"/>
+			<origin xyz="0.033599981 0 0" rpy="0 ${radians(90)} 0"/>
 			<parent link="$(arg 6th_link_name)"/>
 			<child link="${child}"/>
